File: EAGLE/Deployment/subscale_deployment.brd (EAGLE design)
At the start: 55.9 x 50.8 mm, 9 parts, among them J1 FEMALE 2x3, Q1 100V 14A

Commit message: It almost works
Other:
- board size 55.9 x 50.8 mm -> 56.9 x 50.8 mm
- board text added: "+"
- board text added: "3V3"
- board text added: "9V Battery"
- board text added: "Beep"
- board text added: "CS"
- board text added: "DRAIN"
- board text added: "E-Match"
- board text added: "GATE"
- board text added: "GND"
- board text added: "MISO"
- board text added: "MOSI"
- board text added: "NC"
- board text added: "RESET"
- board text added: "SCK"
- board text added: "SRC"
- board text added: "Screw Switch"
- board text added: "–"
Changed lines of the file:
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@@
 <layer number="23" name="tOrigins" color="15" fill="1" visible="yes" active="yes"/>
 <layer number="24" name="bOrigins" color="15" fill="1" visible="yes" active="yes"/>
-<layer number="25" name="tNames" color="7" fill="1" visible="yes" active="yes"/>
-<layer number="26" name="bNames" color="7" fill="1" visible="yes" active="yes"/>
-<layer number="27" name="tValues" color="7" fill="1" visible="yes" active="yes"/>
-<layer number="28" name="bValues" color="7" fill="1" visible="yes" active="yes"/>
+<layer number="25" name="tNames" color="7" fill="1" visible="no" active="yes"/>
+<layer number="26" name="bNames" color="7" fill="1" visible="no" active="yes"/>
+<layer number="27" name="tValues" color="7" fill="1" visible="no" active="yes"/>
+<layer number="28" name="bValues" color="7" fill="1" visible="no" active="yes"/>
 <layer number="29" name="tStop" color="7" fill="3" visible="no" active="yes"/>
 <layer number="30" name="bStop" color="7" fill="6" visible="no" active="yes"/>
@@
 <board>
 <plain>
-<wire x1="7.62" y1="0" x2="63.5" y2="0" width="0" layer="20"/>
+<wire x1="6.604" y1="0" x2="63.5" y2="0" width="0" layer="20"/>
 <wire x1="63.5" y1="0" x2="63.51" y2="50.8" width="0" layer="20"/>
-<wire x1="63.51" y1="50.8" x2="7.62" y2="50.8" width="0" layer="20"/>
-<wire x1="7.62" y1="50.8" x2="7.62" y2="0" width="0" layer="20"/>
+<wire x1="63.51" y1="50.8" x2="6.604" y2="50.8" width="0" layer="20"/>
+<wire x1="6.604" y1="50.8" x2="6.604" y2="0" width="0" layer="20"/>
 <hole x="49.71" y="5.93" drill="3.1"/>
 <hole x="52.97" y="42.07" drill="3.1"/>
 <hole x="19.66" y="20.25" drill="3.1"/>
+<text x="38.735" y="38.1" size="1.5" layer="21">9V Battery</text>
+<text x="24.511" y="39.751" size="1.5" layer="21">Screw Switch</text>
+<text x="36.83" y="7.239" size="1.5" layer="21">E-Match
+</text>
+<text x="25.273" y="12.065" size="1.5" layer="21">Beep</text>
+<text x="39.878" y="40.005" size="2" layer="21">+</text>
+<text x="45.085" y="40.259" size="2" layer="21">–</text>
+<text x="24.511" y="9.398" size="2" layer="21">+</text>
+<text x="29.718" y="9.652" size="2" layer="21">–</text>
+<text x="15.494" y="47.498" size="0.7" layer="21" rot="R90">GND</text>
+<text x="18.161" y="47.498" size="0.7" layer="21" rot="R90">MOSI</text>
+<text x="20.701" y="47.498" size="0.7" layer="21" rot="R90">3V3</text>
+<text x="15.494" y="37.973" size="0.7" layer="21" rot="R90">RESET</text>
+<text x="18.034" y="39.243" size="0.7" layer="21" rot="R90">SCK</text>
+<text x="20.574" y="38.862" size="0.7" layer="21" rot="R90">MISO</text>
+<text x="8.636" y="5.969" size="0.7" layer="21">SRC</text>
+<text x="7.62" y="3.556" size="0.7" layer="21">DRAIN</text>
+<text x="8.001" y="8.509" size="0.7" layer="21">GATE</text>
+<text x="9.271" y="15.367" size="0.7" layer="21">NC</text>
+<text x="9.017" y="18.034" size="0.7" layer="21">3V3</text>
+<text x="8.763" y="20.574" size="0.7" layer="21">GND</text>
+<text x="8.89" y="23.114" size="0.7" layer="21">SCK</text>
+<text x="8.382" y="25.654" size="0.7" layer="21">MISO</text>
+<text x="8.255" y="28.194" size="0.7" layer="21">MOSI</text>
+<text x="9.525" y="30.607" size="0.7" layer="21">CS</text>
+<text x="9.525" y="33.147" size="0.7" layer="21">NC</text>
 </plain>
 <attributes>
@@
 <contactref element="J5" pad="4"/>
 <contactref element="J1" pad="5"/>
-<wire x1="27.94" y1="15.24" x2="22.351" y2="20.829" width="0.25" layer="16"/>
-<wire x1="22.351" y1="20.829" x2="22.351" y2="21.36465" width="0.25" layer="16"/>
-<wire x1="22.351" y1="21.36465" x2="17.68065" y2="26.035" width="0.25" layer="16"/>
+<wire x1="27.94" y1="15.24" x2="27.94" y2="15.77565" width="0.25" layer="16"/>
+<wire x1="27.94" y1="15.77565" x2="17.68065" y2="26.035" width="0.25" layer="16"/>
 <wire x1="17.68065" y1="26.035" x2="12.7" y2="26.035" width="0.25" layer="16"/>
 <wire x1="12.7" y1="26.035" x2="12.7" y2="26.09161875" width="0.25" layer="16"/>
@@
 </drawing>
 <compatibility>
+<note version="6.3" minversion="6.2.2" severity="warning">
+Since Version 6.2.2 text objects can contain more than one line,
+which will not be processed correctly with this version.
+</note>
 <note version="8.2" severity="warning">
 Since Version 8.2, EAGLE supports online libraries. The ids
